Commit message: [Qilin][gazebo] Add launch file and gazebo environment

File: robots/uav.urdf.xacro (robot description, xacro)
@@ -4,15 +4,15 @@
   <!-- robot urdf -->
   <xacro:include filename="$(find mini_quadrotor)/urdf/robot.urdf.xacro" />
-  <!-- additional model -->
-  <xacro:extra_module name = "Apriltag_frame" parent = "main_body">
-    <origin xyz=" 0.173 0.00 -0.008" rpy="0 ${pi} 0"/>
-    <inertial>
-      <mass value = "0.00001" />
-      <origin xyz="0 0 0" rpy="0 0 0"/>
-      <inertia
-          ixx="0.000001" ixy="0.0" ixz="0.0"
-          iyy="0.000001" iyz="0.0"
-          izz="0.000002"/>
-    </inertial>
-  </xacro:extra_module>
+  <!-- <!-\- additional model -\-> -->
+  <!-- <xacro:extra_module name = "Apriltag_frame" parent = "main_body"> -->
+  <!--   <origin xyz=" 0.173 0.00 -0.008" rpy="0 ${pi} 0"/> -->
+  <!--   <inertial> -->
+  <!--     <mass value = "0.00001" /> -->
+  <!--     <origin xyz="0 0 0" rpy="0 0 0"/> -->
+  <!--     <inertia -->
+  <!--         ixx="0.000001" ixy="0.0" ixz="0.0" -->
+  <!--         iyy="0.000001" iyz="0.0" -->
+  <!--         izz="0.000002"/> -->
+  <!--   </inertial> -->
+  <!-- </xacro:extra_module> -->
 </robot>
