Commit message: [Qilin]{store]

File: urdf/camera.xacro (robot description, xacro)
@@ -22,5 +22,5 @@
   <!-- upward camera: depth, color based on left camera -->
   <xacro:extra_module name = "upward_camera_frame" parent = "trunk">
-    <origin xyz="0.0925 0.00 0.1" rpy="0 ${-pi / 2} 0"/>
+    <origin xyz="0.270 0.00 0.137" rpy="0 ${-pi / 2} 0"/>
     <inertial>
       <mass value = "0.00001" />

Commit message: [Qilin][simulation] Add a apriltag
There is a problem. I can see apriltag in rviz but cannot see in gazebo.

File: urdf/camera.xacro (robot description, xacro)
@@ -43,4 +43,36 @@
     </inertial>
   </xacro:extra_module>
+    <!-- New link for the AprilTag -->
+  <link name="apriltag_link">
+    <gazebo reference="apriltag_link">
+      <material>Apriltag36_11_00000</material>
+    </gazebo>
+    <visual>
+      <origin xyz="0 0 0" rpy="${-pi} 0 0"/>
+      <geometry>
+        <box size="0.032 0.032 0.001"/>
+      </geometry>
+      <material name="apriltag_material">
+        <texture filename="package://cooperation_landing/gazebo_model/models/Apriltag36_11_00000/materials/textures/tag36_11_00000.png"/>
+      </material>
+    </visual>
+    <collision>
+      <origin xyz="0 0 0" rpy="0 0 0"/>
+      <geometry>
+        <box size="0.032 0.032 0.001"/>
+      </geometry>
+    </collision>
+    <inertial>
+      <mass value="0.01"/>
+      <origin xyz="0 0 0"/>
+      <inertia ixx="0.0001" ixy="0.0" ixz="0.0" iyy="0.0001" iyz="0.0" izz="0.0001"/>
+    </inertial>
+  </link>
+  <!-- Add a joint to attach the AprilTag to the drone -->
+  <joint name="apriltag_joint" type="fixed">
+    <parent link="trunk"/>
+    <child link="apriltag_link"/>
+    <origin xyz="0.2 0 0.2"/>
+  </joint>
   <!-- PROPERTY-->
   <gazebo reference="upward_camera_frame">

Commit message: [Qilin][simulation] Mount the apriltag on the drone
Use the blender to create a cube which texture is a Apriltag. And then the picture of apriltag can be seen in gazebo.

File: urdf/camera.xacro (robot description, xacro)
@@ -22,5 +22,5 @@
   <!-- upward camera: depth, color based on left camera -->
   <xacro:extra_module name = "upward_camera_frame" parent = "trunk">
-    <origin xyz="0.270 0.00 0.137" rpy="0 ${-pi / 2} 0"/>
+    <origin xyz="0.270 0.00 0.137" rpy="0 ${-pi / 2} ${-pi / 2}"/>
     <inertial>
       <mass value = "0.00001" />
@@ -43,36 +43,4 @@
     </inertial>
   </xacro:extra_module>
-    <!-- New link for the AprilTag -->
-  <link name="apriltag_link">
-    <gazebo reference="apriltag_link">
-      <material>Apriltag36_11_00000</material>
-    </gazebo>
-    <visual>
-      <origin xyz="0 0 0" rpy="${-pi} 0 0"/>
-      <geometry>
-        <box size="0.032 0.032 0.001"/>
-      </geometry>
-      <material name="apriltag_material">
-        <texture filename="package://cooperation_landing/gazebo_model/models/Apriltag36_11_00000/materials/textures/tag36_11_00000.png"/>
-      </material>
-    </visual>
-    <collision>
-      <origin xyz="0 0 0" rpy="0 0 0"/>
-      <geometry>
-        <box size="0.032 0.032 0.001"/>
-      </geometry>
-    </collision>
-    <inertial>
-      <mass value="0.01"/>
-      <origin xyz="0 0 0"/>
-      <inertia ixx="0.0001" ixy="0.0" ixz="0.0" iyy="0.0001" iyz="0.0" izz="0.0001"/>
-    </inertial>
-  </link>
-  <!-- Add a joint to attach the AprilTag to the drone -->
-  <joint name="apriltag_joint" type="fixed">
-    <parent link="trunk"/>
-    <child link="apriltag_link"/>
-    <origin xyz="0.2 0 0.2"/>
-  </joint>
   <!-- PROPERTY-->
   <gazebo reference="upward_camera_frame">
@@ -100,5 +68,5 @@
         <alwaysOn>true</alwaysOn>
         <updateRate>0.0</updateRate>
-        <cameraName>upword_camera</cameraName>
+        <cameraName>upward_camera</cameraName>
         <imageTopicName>image_raw</imageTopicName>
         <cameraInfoTopicName>camera_info</cameraInfoTopicName>

Commit message: [Qilin]{simulation} change the camera's frame and pixel

File: urdf/camera.xacro (robot description, xacro)
@@ -33,5 +33,5 @@
   </xacro:extra_module>
   <xacro:extra_module name = "upward_camera_optical_frame" parent = "upward_camera_frame">
-    <origin xyz="0 0 0" rpy="0 0 0"/>
+    <origin xyz="0 0 0" rpy="${-pi / 2} 0 0"/>
     <inertial>
      <mass value = "0.00001" />
@@ -44,5 +44,5 @@
   </xacro:extra_module>
   <!-- PROPERTY-->
-  <gazebo reference="upward_camera_frame">
+  <gazebo reference="upward_camera_optical_frame">
     <sensor type="camera" name="upward_camera">
       <update_rate>30.0</update_rate>
@@ -50,5 +50,5 @@
         <horizontal_fov>1.57</horizontal_fov>
         <image>
-          <width>1080</width>
+          <width>1280</width>
           <height>720</height>
           <format>RGB</format>
