Commit message: [xuanwu][urdf] Mount a landing gear and change files names

File: urdf/ground_robot.gazebo.xacro (robot description, xacro)
@@ -3,5 +3,5 @@
   <xacro:arg name="robot_name" default="qilin" />
   <!-- robot urdf -->
-  <xacro:include filename="$(find cooperation_landing)/urdf/camera.urdf.xacro" />
+  <xacro:include filename="$(find cooperation_landing)/urdf/ground_robot.urdf.xacro" />
   <gazebo reference="upward_camera_optical_frame">
     <sensor type="camera" name="upward_camera">

File: urdf/ground_robot.urdf.xacro (robot description, xacro)
@@ -43,3 +43,14 @@
     </inertial>
   </xacro:extra_module>
+  <xacro:extra_module name = "landing_gear_frame" parent = "trunk" visible = "1" model_url = "package://cooperation_landing/urdf/mesh/landing_gear.dae">
+    <origin xyz="0.18 0 0.06" rpy="0 0 ${pi/2}"/>
+    <inertial>
+     <mass value = "0.00001" />
+     <origin xyz="0 0 0" rpy="0 0 0"/>
+      <inertia
+          ixx="0.000001" ixy="0.0" ixz="0.0"
+          iyy="0.000001" iyz="0.0"
+          izz="0.000002"/>
+    </inertial>
+  </xacro:extra_module>
 </robot>
