Commit message: [xuanwu][urdf] Add cameras function for aerial and ground robots

File: urdf/aerial_robot.gazebo.xacro (robot description, xacro)
@@ -1,5 +1,5 @@
 <?xml version="1.0"?>
 <robot
-    xmlns:xacro="http://www.ros.org/wiki/xacro" name="mini_quadrotor" >
+    xmlns:xacro="http://www.ros.org/wiki/xacro" name="xuanwu" >
   <xacro:arg name="robot_name" default="quadrotor" />
   <!-- robot urdf -->
@@ -12,3 +12,40 @@
     <mu2>0.1</mu2>
   </gazebo>
+  <gazebo reference="aerial_robot_camera_frame">
+    <sensor type="camera" name="aerial_robot_camera">
+      <update_rate>30.0</update_rate>
+      <camera name="head">
+        <horizontal_fov>1.57</horizontal_fov>
+        <image>
+          <width>1280</width>
+          <height>720</height>
+          <format>RGB</format>
+        </image>
+        <clip>
+          <near>0.02</near>
+          <far>300</far>
+        </clip>
+        <noise>
+          <type>gaussian</type>
+          <mean>0.0</mean>
+          <stddev>0.007</stddev>
+        </noise>
+      </camera>
+      <plugin name="camera_controller" filename="libgazebo_ros_camera.so">
+        <robotNamespace>aerial_robot_camera</robotNamespace>
+        <alwaysOn>true</alwaysOn>
+        <updateRate>0.0</updateRate>
+        <cameraName>aerial_robot_camera</cameraName>
+        <imageTopicName>image_raw</imageTopicName>
+        <cameraInfoTopicName>camera_info</cameraInfoTopicName>
+        <frameName>$(arg robot_name)/aerial_robot_camera_frame</frameName>
+        <hackBaseline>0.07</hackBaseline>
+        <distortionK1>0.0</distortionK1>
+        <distortionK2>0.0</distortionK2>
+        <distortionK3>0.0</distortionK3>
+        <distortionT1>0.0</distortionT1>
+        <distortionT2>0.0</distortionT2>
+      </plugin>
+    </sensor>
+  </gazebo>
 </robot>

File: urdf/aerial_robot.urdf.xacro (robot description, xacro)
@@ -4,4 +4,25 @@
   <!-- robot urdf -->
   <xacro:include filename="$(find xuanwu)/urdf/robot.urdf.xacro" />
+  <!-- camera -->
+  <xacro:extra_module name = "aerial_robot_camera_frame" parent = "main_body" visible = "0" >
+    <origin xyz="-0.058 0 -0.047" rpy="0 0 ${pi}"/>
+    <inertial>
+      <mass value = "0.00001" />
+      <origin xyz="0 0 0" rpy="0 0 0"/>
+      <inertia
+          ixx="0.0" ixy="0.0" ixz="0.0"
+          iyy="0.0" iyz="0.0" izz="0.0"/>
+    </inertial>
+  </xacro:extra_module>
+  <xacro:extra_module name = "aerial_robot_camera_optical_frame" parent = "aerial_robot_camera_frame" visible = "0" >
+    <origin xyz="0 0 0" rpy="${-pi/2} 0 ${pi/2}"/>
+    <inertial>
+      <mass value = "0.00001" />
+      <origin xyz="0 0 0" rpy="0 0 0"/>
+      <inertia
+          ixx="0.0" ixy="0.0" ixz="0.0"
+          iyy="0.0" iyz="0.0" izz="0.0"/>
+    </inertial>
+  </xacro:extra_module>
   <!-- <!-\- additional model -\-> -->
   <joint name="apriltag_0_joint" type="fixed">

File: urdf/ground_robot.gazebo.xacro (robot description, xacro)
@@ -4,6 +4,6 @@
   <!-- robot urdf -->
   <xacro:include filename="$(find cooperation_landing)/urdf/ground_robot.urdf.xacro" />
-  <gazebo reference="upward_camera_optical_frame">
-    <sensor type="camera" name="upward_camera">
+  <gazebo reference="ground_robot_camera_frame">
+    <sensor type="camera" name="ground_robot_camera">
       <update_rate>30.0</update_rate>
       <camera name="head">
@@ -25,11 +25,11 @@
       </camera>
       <plugin name="camera_controller" filename="libgazebo_ros_camera.so">
-        <robotNamespace>unitree_camera</robotNamespace>
+        <robotNamespace>ground_robot_camera</robotNamespace>
         <alwaysOn>true</alwaysOn>
         <updateRate>0.0</updateRate>
-        <cameraName>upward_camera</cameraName>
+        <cameraName>ground_robot_camera</cameraName>
         <imageTopicName>image_raw</imageTopicName>
         <cameraInfoTopicName>camera_info</cameraInfoTopicName>
-        <frameName>$(arg robot_name)/upward_camera_optical_frame</frameName>
+        <frameName>$(arg robot_name)/ground_robot_camera_frame</frameName>
         <hackBaseline>0.07</hackBaseline>
         <distortionK1>0.0</distortionK1>

File: urdf/ground_robot.urdf.xacro (robot description, xacro)
@@ -21,6 +21,6 @@
   </xacro:macro>
   <!-- upward camera: monocular camera-->
-  <xacro:extra_module name = "upward_camera_frame" parent = "trunk" visible = "0">
-    <origin xyz="${0.270} ${0.00} ${0.137}" rpy="0 ${-pi / 2} ${-pi / 2}"/>
+  <xacro:extra_module name = "ground_robot_camera_frame" parent = "landing_gear" visible = "0">
+    <origin xyz="0 -0.04975 ${0.122}" rpy=" ${pi/2} ${-pi/2} 0"/>
     <inertial>
       <mass value = "0.00001" />
@@ -32,6 +32,6 @@
     </inertial>
   </xacro:extra_module>
-  <xacro:extra_module name = "upward_camera_optical_frame" parent = "upward_camera_frame" visible = "0">
-    <origin xyz="0 0 0" rpy="${-pi / 2} 0 0"/>
+  <xacro:extra_module name = "ground_robot_camera_optical_frame" parent = "ground_robot_camera_frame" visible = "0">
+    <origin xyz="0 0 0" rpy="${-pi/2} 0 ${pi/2}"/>
     <inertial>
      <mass value = "0.00001" />
