Commit message: [xuanwu][urdf] Split landing gear to two parts and add two bricks models

File: urdf/brick_bottom_spawn.xacro (robot description, xacro)
@@ -17,7 +17,7 @@
     </visual>
     <collision>
-      <origin xyz="0 0 0.02"/>
+      <origin xyz="0 0 0.10"/>
       <geometry>
-        <box size="0.01 0.01 0.01"/>
+        <box size="0.15 0.15 0.2"/>
       </geometry>
     </collision>

File: urdf/ground_robot.urdf.xacro (robot description, xacro)
@@ -65,7 +65,13 @@
     </visual>
     <collision>
-      <origin xyz="0 -0.1 0.154"/>
+      <origin xyz="0.2 -0.1 0.154"/>
       <geometry>
-        <box size="0.5 0.5 0.01"/>
+        <box size="0.1 0.5 0.01"/>
+      </geometry>
+    </collision>
+    <collision>
+      <origin xyz="-0.2 -0.1 0.154"/>
+      <geometry>
+        <box size="0.1 0.5 0.01"/>
       </geometry>
     </collision>
