Commit message: [xuanwu][urdf] update simulation env

File: urdf/brick_spawn.xacro (robot description, xacro)
@@ -6,7 +6,7 @@
       <origin xyz="0 0 0.01556" rpy="0 0 0"/>
       <inertia
-          ixx="0.00001" ixy="0" ixz="0"
-          iyy="0.0001" iyz="0"
-          izz="0.0001"/>
+          ixx="0.000001" ixy="0" ixz="0"
+          iyy="0.000001" iyz="0"
+          izz="0.00001"/>
     </inertial>
     <visual>
@@ -16,10 +16,4 @@
       </geometry>
     </visual>
-    <collision>
-      <origin xyz="0 0 0.02"/>
-      <geometry>
-        <box size="0.01 0.01 0.01"/>
-      </geometry>
-    </collision>
   </link>
 </robot>

File: urdf/cube_spawn_put.xacro (robot description, xacro)
@@ -11,5 +11,5 @@
     </inertial>
     <visual>
-      <origin rpy="0 0 0" xyz="0 0 0"/>
+      <origin rpy="${pi/2} 0 0" xyz="0 0.6 0.15"/>
       <geometry>
         <mesh filename="package://cooperation_landing/urdf/mesh/cube_0.3_0.3_1.2.dae" />
@@ -17,7 +17,7 @@
     </visual>
     <collision>
-      <origin xyz="0 0 0.6"/>
+      <origin rpy="0 0 ${pi/2}" xyz="0 0 0.1"/>
       <geometry>
-        <box size="0.3 0.3 1.2"/>
+        <box size="1.2 0.3 0.5"/>
       </geometry>
     </collision>
@@ -26,5 +26,5 @@
     <parent link="cube_put"/>
     <child link="apriltag_12"/>
-    <origin xyz="-0.15 0 0.6" rpy="${pi/2} 0 ${-pi/2}" />
+    <origin xyz="-0.15 0 0.15" rpy="${pi/2} 0 ${-pi/2}" />
     <axis xyz="0 0 1"/>
   </joint>
