Commit message: [xuanwu][urdf] Add collision of landing gear

File: urdf/ground_robot.urdf.xacro (robot description, xacro)
@@ -43,14 +43,31 @@
     </inertial>
   </xacro:extra_module>
-  <xacro:extra_module name = "landing_gear_frame" parent = "trunk" visible = "1" model_url = "package://cooperation_landing/urdf/mesh/landing_gear.dae">
-    <origin xyz="0.18 0 0.06" rpy="0 0 ${pi/2}"/>
+  <joint name="root_joint" type="fixed">
+    <parent link="trunk"/>
+    <child link="landing_gear"/>
+    <origin rpy="0 0 ${pi/2}" xyz="0.18 0 0.06"/>
+    <axis xyz="0 0 1"/>
+  </joint>
+  <link name="landing_gear">
     <inertial>
-     <mass value = "0.00001" />
-     <origin xyz="0 0 0" rpy="0 0 0"/>
+      <mass value = "0.00001" />
+      <origin xyz="0 0 0" rpy="0 0 0"/>
       <inertia
-          ixx="0.000001" ixy="0.0" ixz="0.0"
-          iyy="0.000001" iyz="0.0"
-          izz="0.000002"/>
+          ixx="0.000001" ixy="0" ixz="0"
+          iyy="0.000001" iyz="0"
+          izz="0.000001"/>
     </inertial>
-  </xacro:extra_module>
+    <visual>
+      <origin rpy="0 0 0" xyz="0 0 0"/>
+      <geometry>
+        <mesh filename="package://cooperation_landing/urdf/mesh/landing_gear.dae" />
+      </geometry>
+    </visual>
+    <collision>
+      <origin rpy="0 0 0" xyz="0 0 0"/>
+      <geometry>
+        <box size="0.525 0.414 0.1" />
+      </geometry>
+    </collision>
+  </link>
 </robot>

Commit message: [xuanwu][urdf] Change correct collision param of landing gear

File: urdf/ground_robot.urdf.xacro (robot description, xacro)
@@ -46,5 +46,5 @@
     <parent link="trunk"/>
     <child link="landing_gear"/>
-    <origin rpy="0 0 ${pi/2}" xyz="0.18 0 0.06"/>
+    <origin rpy="0 0 ${pi/2}" xyz="0.18 0 0.057"/>
     <axis xyz="0 0 1"/>
   </joint>
@@ -67,5 +67,5 @@
       <origin rpy="0 0 0" xyz="0 0 0"/>
       <geometry>
-        <box size="0.525 0.414 0.1" />
+        <box size="0.525 0.414 0.15452" />
       </geometry>
     </collision>

Commit message: [xuanwu] Attach xuanwu with landing gear in the beginning

File: urdf/ground_robot.urdf.xacro (robot description, xacro)
@@ -51,5 +51,5 @@
   <link name="landing_gear">
     <inertial>
-      <mass value = "0.00001" />
+      <mass value = "0.001" />
       <origin xyz="0 0 0" rpy="0 0 0"/>
       <inertia
@@ -65,9 +65,21 @@
     </visual>
     <collision>
-      <origin rpy="0 0 0" xyz="0 0 0"/>
+      <origin rpy="0 0 0.15452" xyz="0 0 0"/>
       <geometry>
-        <box size="0.525 0.414 0.15452" />
+        <box size="0.525 0.414 0.01" />
+      </geometry>
+    </collision>
+    <collision>
+      <origin xyz="0 0 0.154"/>
+      <geometry>
+        <box size="0.5 0.3 0.01"/>
       </geometry>
     </collision>
   </link>
+  <gazebo reference="landing_gear">
+    <mu1>100</mu1>
+    <mu2>100</mu2>
+    <kp>100000</kp>
+    <kd>1.0</kd>
+  </gazebo>
 </robot>

Commit message: [xuanwu][urdf] Update collision box of landing gear

File: urdf/ground_robot.urdf.xacro (robot description, xacro)
@@ -43,5 +43,5 @@
     </inertial>
   </xacro:extra_module>
-  <joint name="root_joint" type="fixed">
+  <joint name="landing_gear_joint" type="fixed">
     <parent link="trunk"/>
     <child link="landing_gear"/>
@@ -65,13 +65,7 @@
     </visual>
     <collision>
-      <origin rpy="0 0 0.15452" xyz="0 0 0"/>
+      <origin xyz="0 -0.1 0.154"/>
       <geometry>
-        <box size="0.525 0.414 0.01" />
-      </geometry>
-    </collision>
-    <collision>
-      <origin xyz="0 0 0.154"/>
-      <geometry>
-        <box size="0.5 0.3 0.01"/>
+        <box size="0.5 0.5 0.01"/>
       </geometry>
     </collision>

Commit message: [xuanwu][urdf] Make each landing beam be more wider

File: urdf/ground_robot.urdf.xacro (robot description, xacro)
@@ -67,5 +67,5 @@
       <origin xyz="0.2 -0.1 0.154"/>
       <geometry>
-        <box size="0.1 0.5 0.01"/>
+        <box size="0.2 0.5 0.01"/>
       </geometry>
     </collision>
@@ -73,5 +73,5 @@
       <origin xyz="-0.2 -0.1 0.154"/>
       <geometry>
-        <box size="0.1 0.5 0.01"/>
+        <box size="0.2 0.5 0.01"/>
       </geometry>
     </collision>

Commit message: [xuanwu][urdf] update mass and inertia of landing gear

File: urdf/ground_robot.urdf.xacro (robot description, xacro)
@@ -51,10 +51,10 @@
   <link name="landing_gear">
     <inertial>
-      <mass value = "0.001" />
-      <origin xyz="0 0 0" rpy="0 0 0"/>
+      <mass value = "0.626" />
+      <origin xyz="0.02154 0 0.11318" rpy="0 0 ${-pi/2}"/>
       <inertia
-          ixx="0.000001" ixy="0" ixz="0"
-          iyy="0.000001" iyz="0"
-          izz="0.000001"/>
+          ixx="0.01052048067" ixy="0" ixz="0"
+          iyy="0.0107363246" iyz="0"
+          izz="0.01991415212"/>
     </inertial>
     <visual>

Commit message: [xuanwu][urdf] update tail part model

File: urdf/ground_robot.urdf.xacro (robot description, xacro)
@@ -83,3 +83,31 @@
     <kd>1.0</kd>
   </gazebo>
+  <joint name="tail_part_joint" type="fixed">
+    <parent link="trunk"/>
+    <child link="tail_part"/>
+    <origin rpy="0 0 0" xyz="-0.10 0.0 0.057"/>
+    <axis xyz="0 0 1"/>
+  </joint>
+  <link name="tail_part">
+    <inertial>
+      <mass value = "0.001" />
+      <origin xyz="0.0 0.0 0.0" rpy="0 0 0"/>
+      <inertia
+          ixx="0.01" ixy="0" ixz="0"
+          iyy="0.01" iyz="0"
+          izz="0.01"/>
+    </inertial>
+    <visual>
+      <origin rpy="0 0 0" xyz="0 0 0"/>
+      <geometry>
+        <mesh filename="package://cooperation_landing/urdf/mesh/tail_part.dae" />
+      </geometry>
+    </visual>
+    <collision>
+      <origin xyz="0.2 -0.1 0.154"/>
+      <geometry>
+        <box size="0.2 0.5 0.01"/>
+      </geometry>
+    </collision>
+  </link>
 </robot>

Commit message: [xuanwu][urdf] update the landing gear urdf

File: urdf/ground_robot.urdf.xacro (robot description, xacro)
@@ -46,5 +46,5 @@
     <parent link="trunk"/>
     <child link="landing_gear"/>
-    <origin rpy="0 0 ${pi/2}" xyz="0.18 0 0.057"/>
+    <origin rpy="0 0 0" xyz="0.11 0 0.057"/>
     <axis xyz="0 0 1"/>
   </joint>
