Commit message: [xuanwu][scripts] Improve landing control and stall recovery.

File: urdf/ground_robot.urdf.xacro (robot description, xacro)
@@ -46,5 +46,5 @@
     <parent link="trunk"/>
     <child link="landing_gear"/>
-    <origin rpy="0 0 ${pi/2}" xyz="0.18 0 0.057"/>
+    <origin rpy="0 0 -${pi/2}" xyz="-0.18 0 0.057"/>
     <axis xyz="0 0 1"/>
   </joint>
